File: prototype/sound_machine.kicad_pcb (KiCad board)
At the start: 2 copper layers, 75 x 45 mm, 21 parts, among them J1 Conn_01x04, J10 Conn_01x01, J11 Conn_01x01, J12 Conn_01x01, J13 Conn_01x15, J16 Conn_01x15, J2 Conn_01x15, J3 Conn_01x15, J4 Conn_01x08, J5 Audio-Jack-3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

Commit message: Gerbers
Other:
- board text added: "https://github.com/theapi/sound_machine_hardware prototype v1.0.0"
- board text removed: "https://github.com/theapi/sound_machine v1.0.0"
Changed lines of the file:
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@@
     (visible_elements FFFEF77F)
     (pcbplotparams
-      (layerselection 0x00030_80000001)
-      (usegerberextensions false)
+      (layerselection 0x000f0_80000001)
+      (usegerberextensions true)
       (excludeedgelayer true)
       (linewidth 0.100000)
@@
       (outputformat 1)
       (mirror false)
-      (drillshape 1)
+      (drillshape 0)
       (scaleselection 1)
-      (outputdirectory ""))
+      (outputdirectory gerber/))
   )
   (net 0 "")
@@
     (effects (font (size 0.8 0.8) (thickness 0.1)) (justify mirror))
   )
-  (gr_text "https://github.com/theapi/sound_machine  v1.0.0" (at 142.24 107.95) (layer B.SilkS)
+  (gr_text "https://github.com/theapi/sound_machine_hardware\nprototype  v1.0.0" (at 142.748 107.95) (layer B.SilkS)
     (effects (font (size 0.9 0.9) (thickness 0.2)) (justify left mirror))
   )
